File: lampicka.sch (EAGLE design)
At the start: 15 parts, among them IC1 REG1117, J1 DCJ0202

Commit message: lampicka
Parts:
- IC1: SPICEPREFIX (none) -> J
Connections:
- net N$4 renamed TX
- net N$5 renamed RX
- net N$6 renamed GPIO0
Changed lines of the file:
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@@
 <part name="T3" library="transistor" library_urn="urn:adsk.eagle:library:402" deviceset="*-NPN-" device="SOT23-BEC" package3d_urn="urn:adsk.eagle:package:28748/2" technology="MMBT2222ALT1"/>
 <part name="IR1" library="telefunken" library_urn="urn:adsk.eagle:library:383" deviceset="TSOP17*TB1" device="" package3d_urn="urn:adsk.eagle:package:27879/1" technology="30"/>
-<part name="IC1" library="burr-brown" library_urn="urn:adsk.eagle:library:111" deviceset="REG1117" device="" package3d_urn="urn:adsk.eagle:package:4940/1"/>
+<part name="IC1" library="burr-brown" library_urn="urn:adsk.eagle:library:111" deviceset="REG1117" device="" package3d_urn="urn:adsk.eagle:package:4940/1">
+<attribute name="SPICEPREFIX" value="J"/>
+</part>
 <part name="J1" library="con-jack" library_urn="urn:adsk.eagle:library:154" deviceset="DCJ0202" device="" package3d_urn="urn:adsk.eagle:package:7491/1"/>
 <part name="GND1" library="supply1" library_urn="urn:adsk.eagle:library:371" deviceset="GND" device=""/>
@@
 </segment>
 </net>
-<net name="N$4" class="0">
+<net name="TX" class="0">
 <segment>
 <pinref part="U$1" gate="G$1" pin="UTXD"/>
@@
 <junction x="83.82" y="121.92"/>
 <pinref part="R4" gate="G$1" pin="2"/>
-</segment>
-</net>
-<net name="N$5" class="0">
+<label x="88.9" y="127" size="1.778" layer="95"/>
+</segment>
+</net>
+<net name="RX" class="0">
 <segment>
 <pinref part="U$1" gate="G$1" pin="URXD"/>
@@
 <pinref part="R1" gate="G$1" pin="1"/>
 <pinref part="R5" gate="G$1" pin="2"/>
-</segment>
-</net>
-<net name="N$6" class="0">
+<label x="86.36" y="109.22" size="1.778" layer="95"/>
+</segment>
+</net>
+<net name="GPIO0" class="0">
 <segment>
 <wire x1="83.82" y1="93.98" x2="81.28" y2="93.98" width="0.1524" layer="91"/>
@@
 <pinref part="R6" gate="G$1" pin="2"/>
 <junction x="81.28" y="116.84"/>
-</segment>
-</net>
+<label x="83.82" y="114.3" size="1.778" layer="95"/>
+</segment>
+</net>
