File: PCB-LED_lamp_with_IR/PCB-LED_lamp_with_IR.kicad_pcb (KiCad board)
At the start: 2 copper layers, 8 parts, among them J1 Conn_01x02_Male, U1 ESP-01v090, U2 AMS1117-3.3

Commit message: lamp
Parts:
- removed J1: Conn_01x02_Male, Connector_PinHeader_2.54mm:PinHeader_1x02_P2.54mm_Vertical
- U2: footprint TO_SOT_Packages_SMD:SOT-223 -> Package_TO_SOT_SMD:SOT-223-3_TabPin2
- moved C2 4.02 mm to (115.6, 96.5)
- moved U2 1.27 mm to (111.8, 88.9), turned to 270 degrees
- moved R3 0.13 mm to (104.3, 85.1)
Connections:
- net Net-(R1-Pad1) renamed LEDS2
- net Net-(R3-Pad2) renamed LEDS1
- R2 pad 1: Net-(R2-Pad1) -> +3V3
- R2 pad 2: +3V3 -> LEDS3
- U1 pad 6: Net-(R2-Pad1) -> LEDS3
- U1 pad 8: (no net) -> IR
Routing:
- net +3V3: track 5.08 -> 45.8 mm, vias 0 -> 1
- net GNDREF: track 0.00 -> 27.6 mm, vias 0 -> 2
- net LEDS2: track 0.00 -> 9.04 mm, vias 0 -> 1
- net IR: track 0.00 -> 8.95 mm, vias 0 -> 1
- net LEDS1: track 0.00 -> 8.71 mm, vias 0 -> 1
- net +5V: track 0.00 -> 5.34 mm, vias 0 -> 1
- net Net-(R2-Pad1): track 0.00 -> 5.08 mm, vias 0 -> 1
Other:
- net class Default: via_dia 1 -> 1.8; via_drill 0.4 -> 0.8
- net class Power: via_dia 1 -> 1.8; via_drill 0.4 -> 0.8

Commit message: leds
Parts:
- added J1: Conn_01x03_Female, Connector_PinSocket_2.54mm:PinSocket_1x03_P2.54mm_Vertical, F.Cu at (107.3, 82.3)
- added J2: Conn_01x02_Male, Connector_PinSocket_2.54mm:PinSocket_1x02_P2.54mm_Horizontal, F.Cu at (107.6, 90.2)
- added J3: Conn_01x03_Female, Connector_PinSocket_2.54mm:PinSocket_1x03_P2.54mm_Horizontal, F.Cu at (104.0, 95.9)
- moved C1 1.14 mm to (118.2, 88.9)
- moved R3 0.57 mm to (104.8, 85.3)
- turned R2 to 180 degrees
Connections:
- R2 pad 2: LEDS3 -> LEDS1
- R3 pad 2: LEDS1 -> IR
- U1 pad 1: LEDS1 -> IR
- U1 pad 6: LEDS3 -> LEDS1
- U1 pad 8: IR -> LEDS3
Routing:
- net LEDS3: track 0.00 -> 10.2 mm
- net GNDREF: track 27.6 -> 34.5 mm, vias 2 -> 1
- net Net-(R2-Pad1): track 5.08 -> 0.00 mm, vias 1 -> 0
- net LEDS1: track 8.71 -> 6.14 mm, vias 1 -> 0
- net +5V: track 5.34 -> 7.85 mm
- net LEDS2: track 9.04 -> 10.8 mm, vias 1 -> 0
- net +3V3: track 45.8 -> 47.3 mm, vias 1 -> 0
- net IR: track 8.95 -> 10.2 mm, vias 1 -> 0
Other:
- board text added: "+5V"
- board text added: "GND"

Commit message: settings
Parts:
- added J1: +5V, Connector_PinSocket_2.54mm:PinSocket_1x01_P2.54mm_Vertical, F.Cu at (120.8, 83.3)
- added J4: 3V3 PWR, Connector_PinSocket_2.54mm:PinSocket_1x02_P2.54mm_Horizontal, F.Cu at (107.6, 90.2)
- C1, C2: value 10µ -> 470µ
- J2: value Conn_01x02_Male -> GND; footprint Connector_PinSocket_2.54mm:PinSocket_1x02_P2.54mm_Horizontal -> Connector_PinSocket_2.54mm:PinSocket_1x01_P2.54mm_Vertical
- J3: value Conn_01x03_Female -> OUTPUTS
- J5: renamed from J1; value Conn_01x03_Female -> TSOP4836
- R1, R2: value R -> 3K3
- moved J2 13.7 mm to (120.9, 93.5), turned to 0 degrees
Connections:
- net IR renamed /IR
- J2 pad 1: +3V3 -> GNDREF
Routing:
- net GNDREF: vias 1 -> 0
- net +5V: vias 1 -> 0
Other:
- board text removed: "+5V"
- board text removed: "GND"
